File: DRV2605.sch (EAGLE design)
At the start: 104 parts, among them J1 BM06B-SRSS-TB, J2 BM06B-SRSS-TB, J3 BM06B-SRSS-TB, J4 BM06B-SRSS-TB, J5 BM06B-SRSS-TB, U1 DRV2605L, U11 NRF51X22_QFQF, U2 DRV2605L, U3 DRV2605L, U4 DRV2605L, U5 DRV2605L, U6 DRV2605L, U7 DRV2605L, U8 TCA9548APWR, U9 TCA9548APWR, X1 32.768kHz, X2 8MHz, X4 16MHz, X5 32.768kHz

Commit message: NRF done STM in progress
Connections:
- net P0.26/XL1 renamed PH0
- net P0.27/XL2 renamed PH1
- new net PC14: C17.2, U$9.PC14, X1.1
- new net PC15: C18.2, U$9.PC15, X1.2
- net P0.26/XL2: no longer C17.2, U$9.PC14, X1.1
- net P0.27/XL1: no longer C18.2, U$9.PC15, X1.2
Changed lines of the file:
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@@
 <pinref part="U11" gate="U$1" pin="P0.26@45"/>
-</segment>
-<segment>
-<pinref part="X1" gate="X$1" pin="1"/>
-<wire x1="238.76" y1="218.44" x2="243.84" y2="218.44" width="0.1524" layer="91"/>
-<wire x1="243.84" y1="218.44" x2="243.84" y2="215.9" width="0.1524" layer="91"/>
-<pinref part="C17" gate="C$1" pin="2"/>
-<pinref part="U$9" gate="G$1" pin="PC14"/>
-<wire x1="289.56" y1="215.9" x2="248.92" y2="215.9" width="0.1524" layer="91"/>
-<wire x1="248.92" y1="215.9" x2="248.92" y2="218.44" width="0.1524" layer="91"/>
-<wire x1="248.92" y1="218.44" x2="243.84" y2="218.44" width="0.1524" layer="91"/>
-<junction x="243.84" y="218.44"/>
 </segment>
 </net>
@@
 <wire x1="101.6" y1="106.68" x2="101.6" y2="86.36" width="0.1524" layer="91"/>
 </segment>
-<segment>
-<pinref part="X1" gate="X$1" pin="2"/>
-<wire x1="238.76" y1="205.74" x2="243.84" y2="205.74" width="0.1524" layer="91"/>
-<wire x1="243.84" y1="205.74" x2="243.84" y2="208.28" width="0.1524" layer="91"/>
-<pinref part="C18" gate="C$1" pin="2"/>
-<pinref part="U$9" gate="G$1" pin="PC15"/>
-<wire x1="289.56" y1="213.36" x2="248.92" y2="213.36" width="0.1524" layer="91"/>
-<wire x1="248.92" y1="213.36" x2="248.92" y2="205.74" width="0.1524" layer="91"/>
-<wire x1="248.92" y1="205.74" x2="243.84" y2="205.74" width="0.1524" layer="91"/>
-<junction x="243.84" y="205.74"/>
-</segment>
 </net>
 <net name="P0.17" class="0">
@@
 </segment>
 </net>
-<net name="P0.26/XL1" class="0">
+<net name="PH0" class="0">
 <segment>
 <pinref part="X2" gate="X$1" pin="1"/>
@@
 </segment>
 </net>
-<net name="P0.27/XL2" class="0">
+<net name="PH1" class="0">
 <segment>
 <pinref part="X2" gate="X$1" pin="2"/>
@@
 </segment>
 </net>
+<net name="PC14" class="0">
+<segment>
+<pinref part="X1" gate="X$1" pin="1"/>
+<wire x1="238.76" y1="218.44" x2="243.84" y2="218.44" width="0.1524" layer="91"/>
+<wire x1="243.84" y1="218.44" x2="243.84" y2="215.9" width="0.1524" layer="91"/>
+<pinref part="C17" gate="C$1" pin="2"/>
+<pinref part="U$9" gate="G$1" pin="PC14"/>
+<wire x1="289.56" y1="215.9" x2="248.92" y2="215.9" width="0.1524" layer="91"/>
+<wire x1="248.92" y1="215.9" x2="248.92" y2="218.44" width="0.1524" layer="91"/>
+<wire x1="248.92" y1="218.44" x2="243.84" y2="218.44" width="0.1524" layer="91"/>
+<junction x="243.84" y="218.44"/>
+</segment>
+</net>
+<net name="PC15" class="0">
+<segment>
+<pinref part="X1" gate="X$1" pin="2"/>
+<wire x1="238.76" y1="205.74" x2="243.84" y2="205.74" width="0.1524" layer="91"/>
+<wire x1="243.84" y1="205.74" x2="243.84" y2="208.28" width="0.1524" layer="91"/>
+<pinref part="C18" gate="C$1" pin="2"/>
+<pinref part="U$9" gate="G$1" pin="PC15"/>
+<wire x1="289.56" y1="213.36" x2="248.92" y2="213.36" width="0.1524" layer="91"/>
+<wire x1="248.92" y1="213.36" x2="248.92" y2="205.74" width="0.1524" layer="91"/>
+<wire x1="248.92" y1="205.74" x2="243.84" y2="205.74" width="0.1524" layer="91"/>
+<junction x="243.84" y="205.74"/>
+</segment>
+</net>

Commit message: 6DRVs ARM - done; IMU on board
Parts:
- removed I2C10, I2C12, I2C14, I2C2, I2C4, I2C6, I2C8: JUMPER_3PLACE_NO_XTRA_SMALL, yhtomit_jumpers:JUMPER_3PLACE_NO_XTRA_SMALL
- added C32: 0.1uF, rcl:C-USC0402
- added C33, C34: 22pF, rcl:C-USC0402
- added J6: JST_6_PIN_VERTICAL, SparkFun-Connectors:JST_6_PIN_VERTICAL
- added R24: 10k, rcl:R-US_R0402
- added R26, R27: 4.7k, rcl:R-US_R0402
- added R28, R29: 2.2k, rcl:R-US_R0402
- added Y1: 32.768kHz, SparkFun-Clocks:CRYSTAL-32.768KHZSMD-3.2X1.5
- C13: value 1.0uF -> 0.1uF; device SparkFun-Capacitors:1.0UF-16V-10%(0402) -> rcl:C-USC0402
- C14: value 1.0uF -> 0.1uF
- R13, R14: value 2.2k -> 10k; device SparkFun-Resistors:2.2KOHM-1/10W-1%(0603) -> rcl:R-US_R0402
- U7: value DRV2605L -> BNO080; device SparkFun-PowerIC:DRV2605L -> SparkFun-IC-Special-Function:BNO080
- X2: device Nordic_nRF:XTAL_32KHZ -> SparkFun-Clocks:CRYSTALSMD-5X3.2-4PAD
Connections:
- removed net +OUT7: J7.1, U7.OUT+
- removed net -OUT7: J7.2, U7.OUT-
- removed net COMMON_EN: I2C10.3, I2C12.3, I2C14.3, I2C2.3, I2C4.3, I2C6.3, I2C8.3
- removed net EN7: I2C14.2, U7.EN
- removed net IN/TRIG7: U7.IN/TRIG
- new net !BOOT: R24.1, U7.!BOOT
- new net !CS: U7.!H_CS
- new net !INT: U7.!H_INT
- new net !RST: R13.1, U7.!RST
- new net 3.3V: C13.1, C32.1, R13.2, R14.2, R24.2, R26.2, R27.2, R28.2, R29.2, U7.VDD, U7.VDDIO
- new net ADDR/MOSI: R14.1, U7.H_SA0/MOSI
- new net CAP: C14.1, U7.CAP
- new net N$11: U$9.PC2
- new net N$12: U$9.PC3
- new net N$14: C33.1, U7.CLKSEL1, Y1.1
- new net N$8: U$9.PC0
- new net N$9: U$9.PC1
- new net PS0/WAKE: U7.PS0/WAKE
- new net PS1: U7.PS1
- new net SCL/SCK/RX: R28.1, U7.H_SCL/SCLK/RX
- new net SDA/MISO/TX: R29.1, U7.H_SDA/MISO/TX
- new net S_SCL: R27.1, U7.S_SCL
- new net S_SDA: R26.1, U7.S_SDA
- new net TCK: J6.4, U$9.PA14/JTCK
- new net TDI: J6.3, U$9.PA15/JTDI
- new net TDO: J6.2, U$9.PB3/JTDO
- new net TMS: J6.5, U$9.PA13/JTMS
- new net TRST: J6.1, U$9.PB4/JTRST
- net EN1: now also U$9.PB12/I2S2_WS; no longer I2C2.2
- net EN2: now also U$9.PB0; no longer I2C4.2
- net EN3: now also U$9.PC4; no longer I2C6.2
- net EN4: now also U$9.PA6/SPI1_MISO; no longer I2C8.2
- net EN5: now also U$9.PA4/SPI1_NSS; no longer I2C10.2
- net EN6: no longer I2C12.2
- net GND: now also C32.2, C33.2, C34.2, U7.CLKSEL0, U7.GNDIO
- net IN/TRIG1: now also U$9.PB13/I2S2_CK
- net IN/TRIG2: now also U$9.PB1
- net IN/TRIG3: now also U$9.PC5
- net IN/TRIG4: now also U$9.PA7/SPI1_MOSI
- net IN/TRIG5: now also U$9.PA5/SPI1_SCK
- net N$7: now also C34.1, U7.XIN32, Y1.2; no longer C14.1, U7.REG
- net RST: now also J6.6
- net SCL7: no longer R13.1, U7.SCL
- net SDA7: no longer R14.1, U7.SDA
- net VCC: no longer C13.1, I2C10.1, I2C12.1, I2C14.1, I2C2.1, I2C4.1, I2C6.1, I2C8.1, R13.2, R14.2, U7.VDD, U7.VDD/NC
Other:
- note added: "7-Bit I2C Address Jumper"
- note added: "Default, nothing is set. Solder both to GND to use i2C"
- note added: "Interface I2C UART-RVC UART SPI"
- note added: "PS0 0 1 0 1"
- note added: "PS1 0 0 1 1"
- note added: "Supply Voltage: 2.4V-3.6V"
- note added: "alternative = 0x4A"
- note added: "default = 0x4B"
- note added: "unlsolder I2C pullups when using SPI or UART"
- moved on the sheet: C13, C14, C28, R13, R14, R21
